Commit message: Rebase from 'upstream'

File: prbt_support/urdf/prbt.xacro (robot description, xacro)
@@ -30,4 +30,9 @@
   <!-- instantiate the robot -->
   <xacro:prbt prefix="$(arg robot_prefix)" />
+  <link name="world"/>
+  <joint name="world-base_link-fixed" type="fixed">
+    <parent link="world"/>
+    <child link="$(arg robot_prefix)base_link"/>
+  </joint>
   <!-- TCP -->
   <joint name="$(arg robot_prefix)fixed_joint_tcp" type="fixed">

File: prbt_support/urdf/prbt_macro.xacro (robot description, xacro)
@@ -24,4 +24,8 @@
     <!-- robot foot link -->
     <link name="${prefix}base_link">
+        <inertial>
+          <mass value="2.4"/>
+          <inertia ixx="0"  ixy="0"  ixz="0" iyy="0" iyz="0" izz="0" />
+        </inertial>
       <visual>
         <origin xyz="0 0 0" rpy="0 0 0" />
@@ -49,7 +53,7 @@
     <link name="${prefix}link_1">
       <inertial>
-        <origin xyz="-0.00014 0.02783 0.05093" rpy="0 0 0"/>
         <mass value="7.1"/>
-        <inertia ixx="0"  ixy="0"  ixz="0" iyy="0" iyz="0" izz="0" />
+        <origin xyz="0 -0.026 -0.051" />
+        <inertia ixx="3.53e-2" ixy="0" ixz="0" iyy="3.01e-2" iyz="9.04e-3" izz="1.87e-2" />
       </inertial>
       <visual>
@@ -89,7 +93,7 @@
     <link name="${prefix}link_2">
       <inertial>
-        <origin xyz="0.00001 0.16907 0.02464" rpy="0 0 0"/>
-        <mass value="2.4"/>
-        <inertia ixx="0"  ixy="0"  ixz="0" iyy="0" iyz="0" izz="0" />
+        <mass value="1.7"/>
+        <origin xyz="0 0.162 0.134" />
+        <inertia ixx="3.58e-2"  ixy="0"  ixz="0" iyy="3.22e-3" iyz="-1.45e-3" izz="3.66e-2" />
       </inertial>
       <visual name="first">
@@ -123,7 +127,7 @@
     <link name="${prefix}link_3">
       <inertial>
-        <origin xyz="-0.0001 0.04395 -0.02798" rpy="0 0 0"/>
-        <mass value="5.0"/>
-        <inertia ixx="0"  ixy="0"  ixz="0" iyy="0" iyz="0" izz="0" />
+        <mass value="4.8"/>
+        <origin xyz="0 0.043 -0.027" />
+        <inertia ixx="2.06e-2" ixy="0" ixz="0" iyy="1.08e-2" iyz="-5.36e-3" izz="1.63e-2" />
       </inertial>
       <visual>
@@ -163,7 +167,7 @@
     <link name="${prefix}link_4">
       <inertial>
-        <origin xyz="-0.00008 0.06528 0.06149" rpy="0 0 0"/>
-        <mass value="0.7"/>
-        <inertia ixx="0"  ixy="0"  ixz="0" iyy="0" iyz="0" izz="0" />
+        <mass value="0.9"/>
+        <origin xyz="0 -0.061 0.204" />
+        <inertia ixx="6.79e-3" ixy="0" ixz="0" iyy="4.91e-3" iyz="2.67e-3" izz="3.40e-3" />
       </inertial>
       <visual>
@@ -197,7 +201,7 @@
     <link name="${prefix}link_5">
       <inertial>
-        <origin xyz="-0.00026 0.01873 -0.03434" rpy="0 0 0"/>
-        <mass value="2"/>
-        <inertia ixx="0"  ixy="0"  ixz="0" iyy="0" iyz="0" izz="0" />
+        <mass value="2.6"/>
+        <origin xyz="-0.001 0.021 -0.032" />
+        <inertia ixx="7.37e-3" ixy="4.78e-6" ixz="6.00e-5" iyy="5.87e-3" iyz="-1.71e-3" izz="3.96e-3" />
       </inertial>
       <visual>
@@ -249,4 +253,9 @@
     <!-- Flange -->
     <link name="${prefix}flange">
+      <inertial>
+        <mass value="0.02" />
+        <origin xyz="0 0 0" />
+        <inertia ixx="0" ixy="0" ixz="0" iyy="0" iyz="0" izz="0" />
+      </inertial>
       <visual>
         <origin xyz="0 0 0" rpy="0 0 0" />
@@ -276,4 +285,52 @@
       <child link="${prefix}tool0" />
     </joint>
+    <!-- transmissions for gazebo -->
+    <transmission name="${prefix}joint_1_trans">
+      <type>transmission_interface/SimpleTransmission</type>
+      <joint name="${prefix}joint_1">
+        <hardwareInterface>hardware_interface/PositionJointInterface</hardwareInterface>
+      </joint>
+      <actuator name="${prefix}joint_1_motor"/>
+    </transmission>
+    <transmission name="${prefix}joint_2_trans">
+      <type>transmission_interface/SimpleTransmission</type>
+      <joint name="${prefix}joint_2">
+        <hardwareInterface>hardware_interface/PositionJointInterface</hardwareInterface>
+      </joint>
+      <actuator name="${prefix}joint_2_motor"/>
+    </transmission>
+    <transmission name="${prefix}joint_3_trans">
+      <type>transmission_interface/SimpleTransmission</type>
+      <joint name="${prefix}joint_3">
+        <hardwareInterface>hardware_interface/PositionJointInterface</hardwareInterface>
+      </joint>
+      <actuator name="${prefix}joint_3_motor"/>
+    </transmission>
+    <transmission name="${prefix}joint_4_trans">
+      <type>transmission_interface/SimpleTransmission</type>
+      <joint name="${prefix}joint_4">
+        <hardwareInterface>hardware_interface/PositionJointInterface</hardwareInterface>
+      </joint>
+      <actuator name="${prefix}joint_4_motor"/>
+    </transmission>
+    <transmission name="${prefix}joint_5_trans">
+      <type>transmission_interface/SimpleTransmission</type>
+      <joint name="${prefix}joint_5">
+        <hardwareInterface>hardware_interface/PositionJointInterface</hardwareInterface>
+      </joint>
+      <actuator name="${prefix}joint_5_motor"/>
+    </transmission>
+    <transmission name="${prefix}joint_6_trans">
+      <type>transmission_interface/SimpleTransmission</type>
+      <joint name="${prefix}joint_6">
+        <hardwareInterface>hardware_interface/PositionJointInterface</hardwareInterface>
+      </joint>
+      <actuator name="${prefix}joint_6_motor"/>
+    </transmission>
+    <gazebo>
+      <plugin name="gazebo_ros_control" filename="libgazebo_ros_control.so" >
+        <robotNamespace>prbt</robotNamespace>
+      </plugin>
+    </gazebo>
   </xacro:macro>
 </robot>
