Commit message: Imported upstream version '0.4.8' of 'upstream'

File: prbt_support/urdf/prbt_macro.xacro (robot description, xacro)
@@ -47,5 +47,5 @@
       <child link="${prefix}link_1"/>
       <axis xyz="0 0 1"/>
-      <limit effort="370" velocity="1.57" lower="-2.967" upper="2.967"/>
+      <limit effort="370" velocity="1.57" lower="-2.96706" upper="2.96706"/>
       <dynamics damping="15.0" friction="11" />
     </joint>
@@ -88,5 +88,5 @@
       <child link="${prefix}link_2"/>
       <axis xyz="0 0 1"/>
-      <limit effort="370" velocity="1.57" lower="-2.531" upper="2.531"/>
+      <limit effort="370" velocity="1.57" lower="-2.53073" upper="2.53073"/>
       <dynamics damping="12.0" friction="10.0" />
     </joint>
@@ -122,5 +122,5 @@
       <child link="${prefix}link_3"/>
       <axis xyz="0 0 1"/>
-      <limit effort="176" velocity="1.57" lower="-2.356" upper="2.356"/>
+      <limit effort="176" velocity="1.57" lower="-2.35620" upper="2.35620"/>
       <dynamics damping="4.5" friction="4.5" />
     </joint>
@@ -162,5 +162,5 @@
       <child link="${prefix}link_4"/>
       <axis xyz="0 0 1" />
-      <limit effort="176" velocity="1.57" lower="-2.967" upper="2.967"/>
+      <limit effort="176" velocity="1.57" lower="-2.96706" upper="2.96706"/>
       <dynamics damping="4.2" friction="3.8" />
     </joint>
@@ -196,5 +196,5 @@
       <child link="${prefix}link_5"/>
       <axis xyz="0 0 1" />
-      <limit effort="41.6" velocity="1.57" lower="-2.967" upper="2.967" />
+      <limit effort="41.6" velocity="1.57" lower="-2.96706" upper="2.96706" />
       <dynamics damping="1.5" friction="3.5" />
     </joint>
@@ -248,5 +248,5 @@
       <child link="${prefix}flange"/>
       <axis xyz="0 0 1" />
-      <limit effort="20.1" velocity="1.57" lower="-3.124" upper="3.124" />
+      <limit effort="20.1" velocity="1.57" lower="-3.12414" upper="3.12414" />
       <dynamics damping="4.5" friction="7.0" />
     </joint>
@@ -335,4 +335,64 @@
       </plugin>
     </gazebo>
+    <gazebo reference="${prefix}joint_1">
+      <provideFeedback>true</provideFeedback>
+    </gazebo>
+    <gazebo>
+      <plugin name="ft_sensor" filename="libgazebo_ros_ft_sensor.so">
+	<updateRate>100.0</updateRate>
+	<topicName>prbt/ft_sensor/joint_1</topicName>
+	<jointName>${prefix}joint_1</jointName>
+      </plugin>
+    </gazebo>
+    <gazebo reference="${prefix}joint_2">
+      <provideFeedback>true</provideFeedback>
+    </gazebo>
+    <gazebo>
+      <plugin name="ft_sensor" filename="libgazebo_ros_ft_sensor.so">
+	<updateRate>100.0</updateRate>
+	<topicName>prbt/ft_sensor/joint_2</topicName>
+	<jointName>${prefix}joint_2</jointName>
+      </plugin>
+    </gazebo>
+    <gazebo reference="${prefix}joint_3">
+      <provideFeedback>true</provideFeedback>
+    </gazebo>
+    <gazebo>
+      <plugin name="ft_sensor" filename="libgazebo_ros_ft_sensor.so">
+	<updateRate>100.0</updateRate>
+	<topicName>prbt/ft_sensor/joint_3</topicName>
+	<jointName>${prefix}joint_3</jointName>
+      </plugin>
+    </gazebo>
+    <gazebo reference="${prefix}joint_4">
+      <provideFeedback>true</provideFeedback>
+    </gazebo>
+    <gazebo>
+      <plugin name="ft_sensor" filename="libgazebo_ros_ft_sensor.so">
+	<updateRate>100.0</updateRate>
+	<topicName>prbt/ft_sensor/joint_4</topicName>
+	<jointName>${prefix}joint_4</jointName>
+      </plugin>
+    </gazebo>
+    <gazebo reference="${prefix}joint_5">
+      <provideFeedback>true</provideFeedback>
+    </gazebo>
+    <gazebo>
+      <plugin name="ft_sensor" filename="libgazebo_ros_ft_sensor.so">
+	<updateRate>100.0</updateRate>
+	<topicName>prbt/ft_sensor/joint_5</topicName>
+	<jointName>${prefix}joint_5</jointName>
+      </plugin>
+    </gazebo>
+    <gazebo reference="${prefix}joint_6">
+      <provideFeedback>true</provideFeedback>
+    </gazebo>
+    <gazebo>
+      <plugin name="ft_sensor" filename="libgazebo_ros_ft_sensor.so">
+	<updateRate>100.0</updateRate>
+	<topicName>prbt/ft_sensor/joint_6</topicName>
+	<jointName>${prefix}joint_6</jointName>
+      </plugin>
+    </gazebo>
   </xacro:macro>
 </robot>
