Commit message: Imported upstream version '0.5.20' of 'upstream'

File: prbt_moveit_config/config/prbt_manipulator.srdf.xacro (robot description, xacro)
@@ -20,4 +20,12 @@
       <chain base_link="${prefix}base_link" tip_link="${prefix}flange" />
     </group>
+    <group_state name="all-zeros" group="manipulator">
+        <joint name="${prefix}joint_1" value="0" />
+        <joint name="${prefix}joint_2" value="0" />
+        <joint name="${prefix}joint_3" value="0" />
+        <joint name="${prefix}joint_4" value="0" />
+        <joint name="${prefix}joint_5" value="0" />
+        <joint name="${prefix}joint_6" value="0" />
+    </group_state>
     <!--
     DISABLE COLLISIONS: By default it is assumed that any link of the robot could potentially come
